File: kicad/psg14_emu/psg14_emu/psg14_emu.sch (KiCad schematic (older format))
At the start: 4 parts, among them U1 STM32F030F4Px

Commit message: [psg14_emu]
Parts:
- added U?: LTV-847S, Package_DIP:SMDIP-16_W9.53mm, symbol Isolator:LTV-847S
Changed lines of the file:
@@
 EESchema Schematic File Version 4
+LIBS:psg14_emu-cache
 EELAYER 26 0
 EELAYER END
@@
 Text Label 4525 3115 0    50   ~ 0
 GND
+$Comp
+L Isolator:LTV-847S U?
+U 1 1 5BC26E11
+P 7160 2665
+F 0 "U?" H 7160 2990 50  0000 C CNN
+F 1 "LTV-847S" H 7160 2899 50  0000 C CNN
+F 2 "Package_DIP:SMDIP-16_W9.53mm" H 7160 2365 50  0001 C CNN
+F 3 "http://www.us.liteon.com/downloads/LTV-817-827-847.PDF" H 6560 3115 50  0001 C CNN
+	1    7160 2665
+	1    0    0    -1
+$EndComp
 $EndSCHEMATC

Commit message: [psg14_emu] Schematics ready
Parts:
- added C1: 100nF, symbol Device:C_Small
- added D1: LED_GREEN, symbol Device:LED_Small
- added J1: Buttons, symbol Connector_Generic:Conn_01x04
- added J3: Conn_ARM_JTAG_SWD_10, Connector_PinHeader_1.27mm:PinHeader_2x05_P1.27mm_Vertical_SMD, symbol Connector:Conn_ARM_JTAG_SWD_10
- added J4, J5, J6: Conn_01x03, symbol Connector_Generic:Conn_01x03
- added R10, R11, R12, R13, R6, R7, R8, R9: 330, symbol Device:R_Small
- added R3, R4: 10K, symbol Device:R_Small
- added R5: 68, symbol Device:R_Small
- added unit 2 of U2
- added unit 3 of U2
- added unit 1 of U2
- added U3: LTV-847S, Package_DIP:SMDIP-16_W9.53mm, symbol Isolator:LTV-847S
- gave numbers to parts that had none: 2
Connections:
- net labels added: B0, B1, DO0, DO1, DO2, DO3, DO4, DO5, DO6, DO7, GND_O, OUT0, OUT1, OUT2, OUT3, OUT4, OUT5, OUT6, OUT7, SWDCLK, SWDIO
- wire segments 2 -> 8
- no-connect marks 2 -> 4

Commit message: [psg14_emu] Assignements
Parts:
- added J7: Conn_01x02_MountingPin, symbol Connector_Generic_MountingPin:Conn_01x02_MountingPin
- C1: footprint (none) -> Capacitors_SMD:C_0805_HandSoldering
- D1: footprint (none) -> LEDs:LED_D5.0mm
- J1: footprint (none) -> Connectors_Terminal_Blocks:TerminalBlock_bornier-4_P5.08mm
Changed lines of the file:
@@
 F 0 "C1" H 2352 2671 50  0000 L CNN
 F 1 "100nF" H 2352 2580 50  0000 L CNN
-F 2 "" H 2260 2625 50  0001 C CNN
+F 2 "Capacitors_SMD:C_0805_HandSoldering" H 2260 2625 50  0001 C CNN
 F 3 "~" H 2260 2625 50  0001 C CNN
 	1    2260 2625
@@
 F 0 "D1" V 2695 3365 50  0000 R CNN
 F 1 "LED_GREEN" V 2600 3535 50  0000 R CNN
-F 2 "" V 2680 3125 50  0001 C CNN
+F 2 "LEDs:LED_D5.0mm" V 2680 3125 50  0001 C CNN
 F 3 "~" V 2680 3125 50  0001 C CNN
 	1    2680 3125
@@
 F 0 "J1" H 1695 3260 50  0000 C CNN
 F 1 "Buttons" H 1695 3351 50  0000 C CNN
-F 2 "" H 1775 3685 50  0001 C CNN
+F 2 "Connectors_Terminal_Blocks:TerminalBlock_bornier-4_P5.08mm" H 1775 3685 50  0001 C CNN
 F 3 "~" H 1775 3685 50  0001 C CNN
 	1    1775 3685
@@
 Text Label 9400 3660 2    50   ~ 0
 GND_O
+$Comp
+L Connector_Generic_MountingPin:Conn_01x02_MountingPin J7
+U 1 1 5BC638B8
+P 1260 2670
+F 0 "J7" H 1348 2493 50  0000 L CNN
+F 1 "Conn_01x02_MountingPin" H 1348 2584 50  0000 L CNN
+F 2 "" H 1260 2670 50  0001 C CNN
+F 3 "~" H 1260 2670 50  0001 C CNN
+	1    1260 2670
+	-1   0    0    1
+$EndComp
 $EndSCHEMATC

Commit message: [psg14_emu] PCB tracing
Parts:
- removed J7: Conn_01x02_MountingPin, symbol Connector_Generic_MountingPin:Conn_01x02_MountingPin
- added C2: 100nF, Capacitors_SMD:C_0805_HandSoldering, symbol Device:C_Small
- added MH1: BatteryWire, Mounting_Holes:MountingHole_2.5mm, symbol Mechanical:MountingHole
- added MH2, MH3, MH4, MH5: MountingHole, Mounting_Holes:MountingHole_3.2mm_M3, symbol Mechanical:MountingHole
- J2: footprint (none) -> Pin_Headers:Pin_Header_Straight_1x02_Pitch2.54mm
- J3: footprint Connector_PinHeader_1.27mm:PinHeader_2x05_P1.27mm_Vertical_SMD -> Pin_Headers:Pin_Header_Straight_2x05_Pitch1.27mm_SMD
- J4, J5, J6: footprint (none) -> Connectors_Terminal_Blocks:TerminalBlock_bornier-3_P5.08mm
- R1, R10, R11, R12, R13, R2, R3, R4, R5, R6, R7, R8, R9: footprint (none) -> Resistors_SMD:R_0805_HandSoldering
- U1: footprint Package_SO:TSSOP-20_4.4x6.5mm_P0.65mm -> Housings_SSOP:TSSOP-20_4.4x6.5mm_Pitch0.65mm
- U2, U3: footprint Package_DIP:SMDIP-16_W9.53mm -> Housings_DIP:SMDIP-16_W9.53mm_Clearance8mm
Connections:
- wire segments 8 -> 9
