File: kicad/psg14_emu/psg14_emu/psg14_emu.kicad_pcb (KiCad board)
At the start: 2 copper layers, 50 x 70 mm, 30 parts, among them J1 Buttons, J2 Battery, J3 Conn_ARM_JTAG_SWD_10, J4 Conn_01x03, J5 Conn_01x03, J6 Conn_01x03, U1 STM32F030F4Px, U2 LTV-847S, U3 LTV-847S

Commit message: [psg14_emu] Ready for production
Parts:
- moved R1 19.4 mm to (78.4, 58.9), turned to 90 degrees
- moved C1 10.4 mm to (78.3, 53.4), turned to 270 degrees
- moved MH2 5.35 mm to (65.0, 25.1)
- moved MH5 5.35 mm to (65.0, 84.7)
- turned C2 to 270 degrees
Routing:
- net -BATT: track 57.5 -> 166.6 mm, vias 0 -> 4
- net /DO4: track 0.00 -> 80.7 mm, vias 0 -> 2
- net +BATT: track 0.00 -> 66.7 mm
- net /DO5: track 0.00 -> 56.8 mm, vias 0 -> 2
- net /B1: track 0.00 -> 52.3 mm, vias 0 -> 1
- net /DO6: track 0.00 -> 48.3 mm, vias 0 -> 4
- net /B0: track 0.00 -> 47.6 mm, vias 0 -> 1
- net /DO7: track 0.00 -> 41.2 mm, vias 0 -> 2
- net Net-(D1-Pad2): track 0.00 -> 38.7 mm
- net /NRST: track 0.00 -> 26.0 mm, vias 0 -> 2
- net /DO3: track 0.00 -> 12.8 mm
- net /SWDCLK: track 0.00 -> 11.2 mm
- net /SWDIO: track 0.00 -> 10.3 mm
- net /DO1: track 0.00 -> 10.3 mm
- net /DO0: track 0.00 -> 10.1 mm
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- added copper zone on B.Cu, net -BATT
- added copper zone on F.Cu, net /GND_O
Other:
- net class Default: clearance 0.25 -> 0.2
- rule trace_clearance: 0.25 -> 0.2
- board text added: "+"
- board text added: "-"
- board text added: "."
- board text added: "0"
- board text added: "1"
- board text added: "2"
- board text added: "3"
- board text added: "4"
- board text added: "5"
- board text added: "6"
- board text added: "7"
- board text added: "C"
- board text added: "Debug"
- board text added: "G"
- board text added: "G_O"
- board text added: "PSG14A_EMU V 1.0"
- board text added: "S"
- board text added: "Эмулятор ПСГ14А (C) Renault Club Kharkiv V 1.0"
