File: kicad/psg14a_power/ch.sch (KiCad schematic (older format))
At the start: 9 parts

Commit message: [psg14a_power] Ready for replication which does not work ;-)
Parts:
- gave numbers to parts that had none: 9
Changed lines of the file:
@@
 	2560 1490 2560 2520
 $Comp
-L Device:C_Small C?
+L Device:C_Small C2
 U 1 1 5C15D7B1
 P 2560 1390
-AR Path="/5C15D206/5C15D7B1" Ref="C?"  Part="1"
-AR Path="/5C1626A2/5C15D7B1" Ref="C?"  Part="1"
-AR Path="/5C1626A4/5C15D7B1" Ref="C?"  Part="1"
-AR Path="/5C1626A6/5C15D7B1" Ref="C?"  Part="1"
-AR Path="/5C1626A8/5C15D7B1" Ref="C?"  Part="1"
-F 0 "C?" H 2652 1436 50  0000 L CNN
+AR Path="/5C15D206/5C15D7B1" Ref="C2"  Part="1"
+AR Path="/5C1626A2/5C15D7B1" Ref="C4"  Part="1"
+AR Path="/5C1626A4/5C15D7B1" Ref="C6"  Part="1"
+AR Path="/5C1626A6/5C15D7B1" Ref="C8"  Part="1"
+AR Path="/5C1626A8/5C15D7B1" Ref="C10"  Part="1"
+F 0 "C2" H 2652 1436 50  0000 L CNN
 F 1 "1uF 50V" H 2652 1345 50  0000 L CNN
 F 2 "Capacitors_SMD:C_0805_HandSoldering" H 2560 1390 50  0001 C CNN
@@
 Connection ~ 1880 2520
 $Comp
-L Device:R_Small R?
+L Device:R_Small R3
 U 1 1 5C15D7C0
 P 1880 2420
-AR Path="/5C15D206/5C15D7C0" Ref="R?"  Part="1"
-AR Path="/5C1626A2/5C15D7C0" Ref="R?"  Part="1"
-AR Path="/5C1626A4/5C15D7C0" Ref="R?"  Part="1"
-AR Path="/5C1626A6/5C15D7C0" Ref="R?"  Part="1"
-AR Path="/5C1626A8/5C15D7C0" Ref="R?"  Part="1"
-F 0 "R?" H 1939 2466 50  0000 L CNN
+AR Path="/5C15D206/5C15D7C0" Ref="R3"  Part="1"
+AR Path="/5C1626A2/5C15D7C0" Ref="R6"  Part="1"
+AR Path="/5C1626A4/5C15D7C0" Ref="R9"  Part="1"
+AR Path="/5C1626A6/5C15D7C0" Ref="R12"  Part="1"
+AR Path="/5C1626A8/5C15D7C0" Ref="R15"  Part="1"
+F 0 "R3" H 1939 2466 50  0000 L CNN
 F 1 "5k1" H 1939 2375 50  0000 L CNN
 F 2 "Resistors_SMD:R_0805_HandSoldering" H 1880 2420 50  0001 C CNN
@@
 $EndComp
 $Comp
-L Device:LED_Small D?
+L Device:LED_Small D2
 U 1 1 5C15D7C7
 P 1880 2180
-AR Path="/5C15D206/5C15D7C7" Ref="D?"  Part="1"
-AR Path="/5C1626A2/5C15D7C7" Ref="D?"  Part="1"
-AR Path="/5C1626A4/5C15D7C7" Ref="D?"  Part="1"
-AR Path="/5C1626A6/5C15D7C7" Ref="D?"  Part="1"
-AR Path="/5C1626A8/5C15D7C7" Ref="D?"  Part="1"
-F 0 "D?" V 1900 2420 50  0000 R CNN
+AR Path="/5C15D206/5C15D7C7" Ref="D2"  Part="1"
+AR Path="/5C1626A2/5C15D7C7" Ref="D5"  Part="1"
+AR Path="/5C1626A4/5C15D7C7" Ref="D8"  Part="1"
+AR Path="/5C1626A6/5C15D7C7" Ref="D11"  Part="1"
+AR Path="/5C1626A8/5C15D7C7" Ref="D14"  Part="1"
+F 0 "D2" V 1900 2420 50  0000 R CNN
 F 1 "green" V 1840 2410 50  0000 R CNN
 F 2 "LEDs:LED_0805_HandSoldering" V 1880 2180 50  0001 C CNN
@@
 	1980 2080 1880 2080
 $Comp
-L Device:D_Small D?
+L Device:D_Small D3
 U 1 1 5C15D7CF
 P 1980 2180
-AR Path="/5C15D206/5C15D7CF" Ref="D?"  Part="1"
-AR Path="/5C1626A2/5C15D7CF" Ref="D?"  Part="1"
-AR Path="/5C1626A4/5C15D7CF" Ref="D?"  Part="1"
-AR Path="/5C1626A6/5C15D7CF" Ref="D?"  Part="1"
-AR Path="/5C1626A8/5C15D7CF" Ref="D?"  Part="1"
-F 0 "D?" V 1900 2300 50  0000 L CNN
+AR Path="/5C15D206/5C15D7CF" Ref="D3"  Part="1"
+AR Path="/5C1626A2/5C15D7CF" Ref="D6"  Part="1"
+AR Path="/5C1626A4/5C15D7CF" Ref="D9"  Part="1"
+AR Path="/5C1626A6/5C15D7CF" Ref="D12"  Part="1"
+AR Path="/5C1626A8/5C15D7CF" Ref="D15"  Part="1"
+F 0 "D3" V 1900 2300 50  0000 L CNN
 F 1 "UF4007" V 1970 2290 50  0000 L CNN
 F 2 "Diodes_THT:D_DO-41_SOD81_P5.08mm_Vertical_AnodeUp" V 1980 2180 50  0001 C CNN
@@
 	1980 1290 1930 1290
 $Comp
-L Device:D_Zener_Small D?
+L Device:D_Zener_Small D1
 U 1 1 5C15D7E7
 P 1830 1290
-AR Path="/5C15D206/5C15D7E7" Ref="D?"  Part="1"
-AR Path="/5C1626A2/5C15D7E7" Ref="D?"  Part="1"
-AR Path="/5C1626A4/5C15D7E7" Ref="D?"  Part="1"
-AR Path="/5C1626A6/5C15D7E7" Ref="D?"  Part="1"
-AR Path="/5C1626A8/5C15D7E7" Ref="D?"  Part="1"
-F 0 "D?" H 1540 1290 50  0000 C CNN
+AR Path="/5C15D206/5C15D7E7" Ref="D1"  Part="1"
+AR Path="/5C1626A2/5C15D7E7" Ref="D4"  Part="1"
+AR Path="/5C1626A4/5C15D7E7" Ref="D7"  Part="1"
+AR Path="/5C1626A6/5C15D7E7" Ref="D10"  Part="1"
+AR Path="/5C1626A8/5C15D7E7" Ref="D13"  Part="1"
+F 0 "D1" H 1540 1290 50  0000 C CNN
 F 1 "BZX85_C12" H 1530 1210 50  0000 C CNN
 F 2 "Diodes_THT:D_DO-41_SOD81_P5.08mm_Vertical_AnodeUp" V 1830 1290 50  0001 C CNN
@@
 $EndComp
 $Comp
-L Device:C_Small C?
+L Device:C_Small C1
 U 1 1 5C15D7EE
 P 1830 1460
-AR Path="/5C15D206/5C15D7EE" Ref="C?"  Part="1"
-AR Path="/5C1626A2/5C15D7EE" Ref="C?"  Part="1"
-AR Path="/5C1626A4/5C15D7EE" Ref="C?"  Part="1"
-AR Path="/5C1626A6/5C15D7EE" Ref="C?"  Part="1"
-AR Path="/5C1626A8/5C15D7EE" Ref="C?"  Part="1"
-F 0 "C?" V 1810 1170 50  0000 C CNN
+AR Path="/5C15D206/5C15D7EE" Ref="C1"  Part="1"
+AR Path="/5C1626A2/5C15D7EE" Ref="C3"  Part="1"
+AR Path="/5C1626A4/5C15D7EE" Ref="C5"  Part="1"
+AR Path="/5C1626A6/5C15D7EE" Ref="C7"  Part="1"
+AR Path="/5C1626A8/5C15D7EE" Ref="C9"  Part="1"
+F 0 "C1" V 1810 1170 50  0000 C CNN
 F 1 "10nF" V 1890 1170 50  0000 C CNN
 F 2 "Capacitors_SMD:C_0805_HandSoldering" H 1830 1460 50  0001 C CNN
@@
 $EndComp
 $Comp
-L Device:R_Small R?
+L Device:R_Small R2
 U 1 1 5C15D7F5
 P 1840 1680
-AR Path="/5C15D206/5C15D7F5" Ref="R?"  Part="1"
-AR Path="/5C1626A2/5C15D7F5" Ref="R?"  Part="1"
-AR Path="/5C1626A4/5C15D7F5" Ref="R?"  Part="1"
-AR Path="/5C1626A6/5C15D7F5" Ref="R?"  Part="1"
-AR Path="/5C1626A8/5C15D7F5" Ref="R?"  Part="1"
-F 0 "R?" V 1770 1380 50  0000 C CNN
+AR Path="/5C15D206/5C15D7F5" Ref="R2"  Part="1"
+AR Path="/5C1626A2/5C15D7F5" Ref="R5"  Part="1"
+AR Path="/5C1626A4/5C15D7F5" Ref="R8"  Part="1"
+AR Path="/5C1626A6/5C15D7F5" Ref="R11"  Part="1"
+AR Path="/5C1626A8/5C15D7F5" Ref="R14"  Part="1"
+F 0 "R2" V 1770 1380 50  0000 C CNN
 F 1 "10K" V 1870 1380 50  0000 C CNN
 F 2 "Resistors_SMD:R_0805_HandSoldering" H 1840 1680 50  0001 C CNN
@@
 $EndComp
 $Comp
-L Device:R_Small R?
+L Device:R_Small R1
 U 1 1 5C15D7FC
 P 1680 1980
-AR Path="/5C15D206/5C15D7FC" Ref="R?"  Part="1"
-AR Path="/5C1626A2/5C15D7FC" Ref="R?"  Part="1"
-AR Path="/5C1626A4/5C15D7FC" Ref="R?"  Part="1"
-AR Path="/5C1626A6/5C15D7FC" Ref="R?"  Part="1"
-AR Path="/5C1626A8/5C15D7FC" Ref="R?"  Part="1"
-F 0 "R?" H 1739 2026 50  0000 L CNN
+AR Path="/5C15D206/5C15D7FC" Ref="R1"  Part="1"
+AR Path="/5C1626A2/5C15D7FC" Ref="R4"  Part="1"
+AR Path="/5C1626A4/5C15D7FC" Ref="R7"  Part="1"
+AR Path="/5C1626A6/5C15D7FC" Ref="R10"  Part="1"
+AR Path="/5C1626A8/5C15D7FC" Ref="R13"  Part="1"
+F 0 "R1" H 1739 2026 50  0000 L CNN
 F 1 "10K" H 1739 1935 50  0000 L CNN
 F 2 "Resistors_SMD:R_0805_HandSoldering" H 1680 1980 50  0001 C CNN
@@
 Connection ~ 1680 1880
 $Comp
-L Transistor_FET:IRF9540N Q?
+L Transistor_FET:IRF9540N Q1
 U 1 1 5C15D806
 P 1880 1880
-AR Path="/5C15D206/5C15D806" Ref="Q?"  Part="1"
-AR Path="/5C1626A2/5C15D806" Ref="Q?"  Part="1"
-AR Path="/5C1626A4/5C15D806" Ref="Q?"  Part="1"
-AR Path="/5C1626A6/5C15D806" Ref="Q?"  Part="1"
-AR Path="/5C1626A8/5C15D806" Ref="Q?"  Part="1"
-F 0 "Q?" H 2085 1834 50  0000 L CNN
+AR Path="/5C15D206/5C15D806" Ref="Q1"  Part="1"
+AR Path="/5C1626A2/5C15D806" Ref="Q2"  Part="1"
+AR Path="/5C1626A4/5C15D806" Ref="Q3"  Part="1"
+AR Path="/5C1626A6/5C15D806" Ref="Q4"  Part="1"
+AR Path="/5C1626A8/5C15D806" Ref="Q5"  Part="1"
+F 0 "Q1" H 2085 1834 50  0000 L CNN
 F 1 "IRF9Z24N" H 2085 1925 50  0000 L CNN
 F 2 "TO_SOT_Packages_THT:TO-220-3_Vertical" H 2080 1805 50  0001 L CIN
