File: kicad/psg14a_power/psg14a_power.kicad_pcb (KiCad board)
At the start: 2 copper layers, 48 parts, among them J1 Power, J2 In, J3 Out, Q1 IRF9Z24N, Q2 IRF9Z24N, Q3 IRF9Z24N, Q4 IRF9Z24N, Q5 IRF9Z24N

Commit message: [psg14a_power]Ready for review by Ioan the Greatest
Parts:
- added D16: green, LEDs:LED_0805_HandSoldering, F.Cu at (104.0, 79.0)
- added H1: Mech, Mounting_Holes:MountingHole_3.2mm_M3, F.Cu at (110.0, 81.0)
- added H2: Mech, Mounting_Holes:MountingHole_3.2mm_M3, F.Cu at (30.0, 81.0)
- added H3: Mech, Mounting_Holes:MountingHole_3.2mm_M3, F.Cu at (110.0, 45.0)
- added R16: 5K1, Resistors_SMD:R_0805_HandSoldering, F.Cu at (101.0, 79.0)
Routing:
- net /GND: track 152.8 -> 220.8 mm, vias 0 -> 16
- net /+24V: track 295.2 -> 358.7 mm
- net /Out2: track 21.8 -> 59.6 mm
- net /Out5: track 21.8 -> 55.8 mm
- net /Out3: track 21.8 -> 45.9 mm
- net /Out4: track 21.8 -> 44.5 mm
- net /Out1: track 82.3 -> 78.7 mm
- net /In5: track 68.6 -> 72.0 mm
- net Net-(D16-Pad1): track 0.00 -> 3.00 mm
- added copper zone on B.Cu, net /GND
- added copper zone on F.Cu, net /GND
- added copper zone on B.Cu, net /Out3
Other:
- board outline added: 88 x 46 mm
- board text added: "V 1.0"
- board text added: "Эмулятор ПСГ14А Renault Club Kharkiv (C) 2018"

Commit message: [Psg14a_power] Ioan the Greatest was drunk. Ready for production
Parts:
- J1: footprint TerminalBlocks_Phoenix:TerminalBlock_Phoenix_MPT-2.54mm_2pol -> TerminalBlocks_Phoenix:TerminalBlock_Phoenix_PT-3.5mm_2pol
Routing:
- net /+24V: track 358.7 -> 352.7 mm
- net /GND: track 220.8 -> 217.7 mm
- removed copper zone on B.Cu, net /Out3
Other:
- net class +24 added: clearance 0.2, trace_width 1, via_dia 1, via_drill 0.5
- board text added: "+"
- board text added: "-"
- board text added: "Входы"
- board text added: "Выходы"
- board text added: "стг пт св 4 5 О"
