File: hw/psg14a_power/ch.kicad_sch (KiCad schematic)
At the start: 9 parts, among them Q2 IRF9Z24N

Commit message: Diode rotated
Changed lines of the file:
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@@
     (stroke (width 0) (type default))
   )
-  (hierarchical_label "Relay_ctl" (shape output) (at 61.468 52.832 0)
+  (hierarchical_label "Relay_ctl" (shape output) (at 61.468 52.832 0) (fields_autoplaced)
     (effects (font (size 1.27 1.27)) (justify left))
   )
-  (hierarchical_label "GND" (shape input) (at 37.846 57.658 180)
+  (hierarchical_label "GND" (shape input) (at 37.846 57.658 180) (fields_autoplaced)
     (effects (font (size 1.27 1.27)) (justify right))
   )
-  (hierarchical_label "+24V" (shape input) (at 65.024 32.766 0)
+  (hierarchical_label "+24V" (shape input) (at 65.024 32.766 0) (fields_autoplaced)
     (effects (font (size 1.27 1.27)) (justify left))
   )
-  (hierarchical_label "In" (shape input) (at 37.846 52.832 180)
+  (hierarchical_label "In" (shape input) (at 37.846 52.832 180) (fields_autoplaced)
     (effects (font (size 1.27 1.27)) (justify right))
   )
@@
     )
   )
-  (symbol (lib_id "Device:D_Zener_Small") (at 46.482 32.766 0) (unit 1)
+  (symbol (lib_id "Device:D_Zener_Small") (at 46.482 32.766 0) (mirror x) (unit 1)
     (in_bom yes) (on_board yes) (dnp no)
-    (property "Reference" "D4" (at 39.116 32.766 0)
+    (property "Reference" "D4" (at 40.64 30.48 0)
       (effects (font (size 1.27 1.27)))
     )
-    (property "Value" "BZX85_C12" (at 38.862 34.798 0)
+    (property "Value" "BZX85_C12" (at 40.64 27.94 0)
       (effects (font (size 1.27 1.27)))
     )
-    (property "Footprint" "Diodes_THT:D_DO-41_SOD81_P5.08mm_Vertical_AnodeUp" (at 46.482 32.766 90)
+    (property "Footprint" "Diodes_THT:D_DO-41_SOD81_P5.08mm_Vertical_AnodeUp" (at 45.212 32.766 90)
       (effects (font (size 1.27 1.27)) hide)
     )
