File: hw/psg14a_power/psg14a_power.kicad_pcb (KiCad board)
At the start: 2 copper layers, 88 x 46 mm, 53 parts, among them J1 Power, J2 In, J3 Out, Q1 IRF9Z24N, Q2 IRF9Z24N, Q3 IRF9Z24N, Q4 IRF9Z24N, Q5 IRF9Z24N

Commit message: Develop/hw (#2)
* Converted to Kicad 7.x 
* Zener diode wrong footprint fixed
Other:
- net class +24 removed
- net class Default removed
